File: Voyager4.kicad_pcb (KiCad board)
At the start: 2 copper layers, 34.9 x 38.1 mm, 33 parts, among them Q1 Q_NPN_BEC, SW1 SW_Push, U1 ATmega32U2-AU, U2 PRTR5V0U2X, Y1 16MHz

Commit message: Prepare for redo
Parts:
- removed C1, C2: 22p, Capacitors_SMD:C_0603
- removed C3: 1uF, Capacitors_SMD:C_0603
- removed C4, C5, CR1, CR2: 0.1u, Capacitors_SMD:C_0603
- removed C6: 4.7u, Capacitors_SMD:C_0603
- removed D18, D9: WS2812B, LEDs:LED_WS2812B-PLCC4
- removed F1: 500mA, Fuse_Holders_and_Fuses:Fuse_SMD1206_Reflow
- removed G***: LOGO, locallib:ai-4.8-ring
- removed MX1, MX2, MX3, MX4: MX-1U, MX_Alps_Hybrid:MX-1U
- removed Q1: Q_NPN_BEC, TO_SOT_Packages_SMD:SOT-23
- removed R1, R5: 10k, Resistors_SMD:R_0805
- removed R10, R27, R7, R8, R9: 1k, Resistors_SMD:R_0805
- removed R2, R3: 22, Resistors_SMD:R_0805
- removed R4, R6: 5.1k, Resistors_SMD:R_0805
- removed SW1: SW_Push, random-keyboard-parts:Jumper-UserFriendly-Small
- removed U1: ATmega32U2-AU, Housings_DFN_QFN:QFN-32-1EP_5x5mm_Pitch0.5mm
- removed U2: PRTR5V0U2X, random-keyboard-parts:SOT143B
- removed USB1: HRO-TYPE-C-31-M-12, Type-C:HRO-TYPE-C-31-M-12-Assembly
- removed Y1: 16MHz, Crystals:Crystal_SMD_3225-4pin_3.2x2.5mm
Routing:
- net GND: track 170.5 -> 0.00 mm, vias 5 -> 0
- net +5V: track 143.5 -> 0.00 mm, vias 6 -> 0
- net ROW0: track 75.5 -> 0.00 mm, vias 1 -> 0
- net LEDGND: track 63.1 -> 0.00 mm, vias 5 -> 0
- net Net-(D18-Pad4): track 61.2 -> 0.00 mm, vias 4 -> 0
- net Net-(R1-Pad2): track 32.6 -> 0.00 mm, vias 4 -> 0
- net VCC: track 29.1 -> 0.00 mm, vias 2 -> 0
- net COL0: track 25.0 -> 0.00 mm, vias 2 -> 0
- net Net-(MX2-Pad4): track 21.5 -> 0.00 mm, vias 1 -> 0
- net Net-(R27-Pad2): track 19.5 -> 0.00 mm, vias 2 -> 0
- net Net-(MX1-Pad4): track 16.4 -> 0.00 mm
- net COL2: track 14.1 -> 0.00 mm, vias 2 -> 0
- net Net-(R4-Pad1): track 13.8 -> 0.00 mm, vias 2 -> 0
- net COL1: track 13.1 -> 0.00 mm, vias 1 -> 0
- net COL3: track 12.5 -> 0.00 mm, vias 2 -> 0
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- removed copper zone on B.Cu, net GND
Other:
- board outline removed
- board text removed: "4"
- board text removed: "R1.0"
- board text removed: "RESET"
- board text removed: "VOYAGER"
- board text removed: "Voyager4"
- board text removed: "kb.ai03.me"

Commit message: Progress
Parts:
- added C1: 22p, Capacitors_SMD:C_0603, B.Cu at (121.9, 75.4)
- added C2: 22p, Capacitors_SMD:C_0603, B.Cu at (118.3, 78.6)
- added C3: 1uF, Capacitors_SMD:C_0603, B.Cu at (121.4, 66.7)
- added C4: 0.1u, Capacitors_SMD:C_0603, B.Cu at (119.9, 70.6)
- added C5: 0.1u, Capacitors_SMD:C_0603, B.Cu at (114.3, 74.2)
- added C6: 4.7u, Capacitors_SMD:C_0603, B.Cu at (121.9, 70.6)
- added D1: SOD-123, Diodes_SMD:D_SOD-123, B.Cu at (57.9, 34.1)
- added D10: SOD-123, Diodes_SMD:D_SOD-123, B.Cu at (96.0, 72.2)
- added D2: SOD-123, Diodes_SMD:D_SOD-123, B.Cu at (77.0, 34.1)
- added D3: SOD-123, Diodes_SMD:D_SOD-123, B.Cu at (96.0, 34.1)
- added D4: SOD-123, Diodes_SMD:D_SOD-123, B.Cu at (57.9, 53.2)
- added D5: SOD-123, Diodes_SMD:D_SOD-123, B.Cu at (77.0, 53.2)
- added D6: SOD-123, Diodes_SMD:D_SOD-123, B.Cu at (96.0, 53.2)
- added D7: SOD-123, Diodes_SMD:D_SOD-123, B.Cu at (100.0, 53.2)
- added D8: SOD-123, Diodes_SMD:D_SOD-123, B.Cu at (57.9, 72.2)
- added D9: SOD-123, Diodes_SMD:D_SOD-123, B.Cu at (77.0, 72.2)
- added F1: 500mA, Fuse_Holders_and_Fuses:Fuse_SMD1206_Reflow, B.Cu at (115.9, 43.7)
- added MX1: MX-1U, MX_Alps_Hybrid:MX-1U, F.Cu at (50.0, 35.7)
- added MX2: MX-1U, MX_Alps_Hybrid:MX-1U, F.Cu at (69.1, 35.7)
- added MX3: MX-1U, MX_Alps_Hybrid:MX-1U, F.Cu at (88.1, 35.7)
- added MX4: MX-1U, MX_Alps_Hybrid:MX-1U, F.Cu at (50.0, 54.8)
- added MX5: MX-1U, MX_Alps_Hybrid:MX-1U, F.Cu at (69.1, 54.8)
- added MX6: MX-1U, MX_Alps_Hybrid:MX-1U, F.Cu at (88.1, 54.8)
- added MX7: MX-1U, MX_Alps_Hybrid:MX-1U, F.Cu at (50.0, 73.8)
- added MX8: MX-1U, MX_Alps_Hybrid:MX-1U, F.Cu at (69.1, 73.8)
- added MX9: MX-1U, MX_Alps_Hybrid:MX-1U, F.Cu at (88.1, 73.8)
- added Q1: Q_NPN_BEC, TO_SOT_Packages_SMD:SOT-23, B.Cu at (108.0, 33.3)
- added R1: 10k, Resistors_SMD:R_0805, B.Cu at (108.0, 77.8)
- added R10: 1k, Resistors_SMD:R_0805, B.Cu at (57.9, 58.7)
- added R11: 1k, Resistors_SMD:R_0805, B.Cu at (77.0, 58.7)
- added R12: 1k, Resistors_SMD:R_0805, B.Cu at (96.0, 58.7)
- added R13: 1k, Resistors_SMD:R_0805, B.Cu at (57.9, 77.8)
- added R14: 1k, Resistors_SMD:R_0805, B.Cu at (77.0, 77.8)
- added R15: 1k, Resistors_SMD:R_0805, B.Cu at (96.0, 77.8)
- added R2: 22, Resistors_SMD:R_0805, B.Cu at (125.4, 69.8)
- added R27: 1k, Resistors_SMD:R_0805, B.Cu at (104.0, 33.3)
- added R3: 22, Resistors_SMD:R_0805, B.Cu at (125.4, 66.7)
- added R4: 5.1k, Resistors_SMD:R_0805, B.Cu at (123.0, 38.9)
- added R5: 10k, Resistors_SMD:R_0805, B.Cu at (107.2, 67.5)
- added R6: 5.1k, Resistors_SMD:R_0805, B.Cu at (114.3, 38.9)
- added R7: 1k, Resistors_SMD:R_0805, B.Cu at (57.9, 39.7)
- added R8: 1k, Resistors_SMD:R_0805, B.Cu at (77.0, 39.7)
- added R9: 1k, Resistors_SMD:R_0805, B.Cu at (96.0, 39.7)
- added SW1: SW_Push, Buttons_Switches_SMD:SW_SPST_SKQG, B.Cu at (102.4, 75.4)
- added SW2: Rotary_Encoder_Switch, Encoder:RotaryEncoder_Alps_EC11E-Switch_Vertical_H20mm, F.Cu at (118.9, 54.8)
- added U1: ATmega32U2-AU, Housings_DFN_QFN:QFN-32-1EP_5x5mm_Pitch0.5mm, B.Cu at (115.1, 68.3)
- added U2: PRTR5V0U2X, random-keyboard-parts:SOT143B, B.Cu at (118.9, 38.6)
- added USB1: HRO-TYPE-C-31-M-12, Type-C:HRO-TYPE-C-31-M-12-Assembly, B.Cu at (118.9, 25.9)
- added Y1: 16MHz, Crystals:Crystal_SMD_3225-4pin_3.2x2.5mm, B.Cu at (118.3, 75.4)
Routing:
- net LEDGND: track 0.00 -> 128.0 mm
- net GND: track 0.00 -> 99.6 mm, vias 0 -> 2
- net +5V: track 0.00 -> 54.6 mm, vias 0 -> 3
- net Net-(R2-Pad2): track 0.00 -> 46.8 mm, vias 0 -> 2
- net ROW1: track 0.00 -> 45.9 mm
- net Net-(R3-Pad1): track 0.00 -> 45.8 mm, vias 0 -> 2
- net ROW2: track 0.00 -> 41.9 mm
- net ROW0: track 0.00 -> 41.9 mm
- net Net-(R1-Pad2): track 0.00 -> 28.4 mm, vias 0 -> 2
- net VCC: track 0.00 -> 19.2 mm, vias 0 -> 2
- net SW10_ROW: track 0.00 -> 14.2 mm
- net Net-(C1-Pad1): track 0.00 -> 11.7 mm
- net Net-(C2-Pad1): track 0.00 -> 9.80 mm
- net D+: track 0.00 -> 7.73 mm
- net D-: track 0.00 -> 7.32 mm
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Other:
- board outline added: 91 x 55 mm
