File: Voyager4.kicad_pcb (KiCad board)
At the start: 2 copper layers, 34.9 x 38.1 mm, 33 parts, among them Q1 Q_NPN_BEC, SW1 SW_Push, U1 ATmega32U2-AU, U2 PRTR5V0U2X, Y1 16MHz

Commit message: Repair project, rev 2.0
Parts:
- removed G***: LOGO, locallib:ai-4.8-ring
- U1: value ATmega32U2-AU -> ATmega32U2-MU
Connections:
- U1 pad 14: Net-(U1-Pad14) -> ROW0
- U1 pad 33: (no net) -> GND
Routing:
- net GND: track 170.5 -> 175.6 mm
- net ROW0: track 75.5 -> 80.1 mm, vias 1 -> 2
Other:
- board text added: "R2.0"
- board text removed: "R1.0"
