File: Voyager4.sch (KiCad schematic (older format))
At the start: 32 parts, among them Q1 Q_NPN_BEC, SW1 SW_Push, U1 ATmega32U2-AU, U2 PRTR5V0U2X, Y1 16MHz

Commit message: Prepare for redo
Parts:
- removed CR1, CR2: 0.1u, Capacitors_SMD:C_0603, symbol Device:C_Small
- removed D18, D9: WS2812B, LEDs:LED_WS2812B-PLCC4, symbol LED:WS2812B
- added D1, D10, D2, D3, D4, D5, D6, D7, D8, D9: SOD-123, Diodes_SMD:D_SOD-123, symbol Device:D_Small
- added MX5, MX6, MX7, MX8, MX9: MX-1U, MX_Alps_Hybrid:MX-1U, symbol MX_Alps_Hybrids:MX-1U
- added R11, R12, R13, R14, R15: 1k, Resistors_SMD:R_0805, symbol Device:R_Small
- added SW2: Rotary_Encoder_Switch, Encoder:RotaryEncoder_Alps_EC11E-Switch_Vertical_H20mm, symbol Device:Rotary_Encoder_Switch
Connections:
- net labels added: ENC_A, ENC_B, ROW1, ROW2, SW10_ROW
- net labels removed: RGBLED
- wire segments 111 -> 133
Other:
- moved on the sheet: F1, R2, R3, R4, R6, U2, USB1

Commit message: Progress
Parts:
- SW1: footprint random-keyboard-parts:Jumper-UserFriendly-Small -> Buttons_Switches_SMD:SW_SPST_SKQG
Changed lines of the file:
@@
 F 0 "SW1" H 1475 1360 50  0000 C CNN
 F 1 "SW_Push" H 1475 1269 50  0000 C CNN
-F 2 "random-keyboard-parts:Jumper-UserFriendly-Small" H 1475 1275 50  0001 C CNN
+F 2 "Buttons_Switches_SMD:SW_SPST_SKQG" H 1475 1275 50  0001 C CNN
 F 3 "" H 1475 1275 50  0001 C CNN
 	1    1475 1075
