File: Voyager4.sch (KiCad schematic (older format))
At the start: 32 parts, among them Q1 Q_NPN_BEC, SW1 SW_Push, U1 ATmega32U2-AU, U2 PRTR5V0U2X, Y1 16MHz

Commit message: Repair project, rev 2.0
Parts:
- removed U1: ATmega32U2-AU, Housings_DFN_QFN:QFN-32-1EP_5x5mm_Pitch0.5mm, symbol MCU_Microchip_ATmega:ATmega32U2-AU
- added U1: ATmega32U2-MU, Housings_DFN_QFN:QFN-32-1EP_5x5mm_Pitch0.5mm, symbol MCU_Microchip_ATmega:ATmega32U2-MU
Connections:
- net +5V: now also U1.31 (UVCC), U1.32 (AVCC), U1.4 (VCC)
- net COL0: now also U1.16 (PB2)
- net COL1: now also U1.25 (PC5)
- net COL2: now also U1.8 (PD2)
- net COL3: now also U1.5 (PC2)
- net D+: now also U1.29 (D+)
- net D-: now also U1.30 (D-)
- net GND: now also Y1.2, Y1.4, U1.28 (UGND), U1.3 (GND), U1.33 (GND)
- net RGBLED: now also U1.9 (PD3)
- net ROW0: now also U1.14 (PB0)
- net at C1.1, Y1.1: now also U1.1 (XTAL1)
- net at C2.1, Y1.3: now also U1.2 (PC0/XTAL2)
- net at R1.2, SW1.2: now also U1.24 (PC1/~RESET)
- net at C3.1: now also U1.27 (UCAP)
- net at R5.2: now also U1.13 (~HWB~/PD7)
- net at R27.2: now also U1.21 (PB7)
Other:
- moved on the sheet: R5
Changed lines of the file:
@@
 EESchema Schematic File Version 4
-LIBS:Voyager6-cache
-EELAYER 26 0
+LIBS:Voyager4-cache
+EELAYER 29 0
 EELAYER END
 $Descr A4 11693 8268
@@
 L Device:R_Small R5
 U 1 1 59E647C2
-P 3975 3000
-F 0 "R5" V 3900 2900 50  0000 L CNN
-F 1 "10k" V 3900 3025 50  0000 L CNN
-F 2 "Resistors_SMD:R_0805" H 3975 3000 50  0001 C CNN
-F 3 "" H 3975 3000 50  0001 C CNN
-	1    3975 3000
+P 3975 3600
+F 0 "R5" V 3900 3500 50  0000 L CNN
+F 1 "10k" V 3900 3625 50  0000 L CNN
+F 2 "Resistors_SMD:R_0805" H 3975 3600 50  0001 C CNN
+F 3 "" H 3975 3600 50  0001 C CNN
+	1    3975 3600
 	0    1    1    0
 $EndComp
@@
 L power:GND #PWR013
 U 1 1 59E64F31
-P 4175 3000
-F 0 "#PWR013" H 4175 2750 50  0001 C CNN
-F 1 "GND" V 4175 2800 50  0000 C CNN
-F 2 "" H 4175 3000 50  0001 C CNN
-F 3 "" H 4175 3000 50  0001 C CNN
-	1    4175 3000
+P 4175 3600
+F 0 "#PWR013" H 4175 3350 50  0001 C CNN
+F 1 "GND" V 4175 3400 50  0000 C CNN
+F 2 "" H 4175 3600 50  0001 C CNN
+F 3 "" H 4175 3600 50  0001 C CNN
+	1    4175 3600
 	0    -1   -1   0
 $EndComp
@@
 	2450 1000 2450 1100
 Wire Wire Line
-	3250 3000 3875 3000
-Wire Wire Line
-	4175 3000 4075 3000
+	3250 3600 3875 3600
+Wire Wire Line
+	4175 3600 4075 3600
 Text Notes 7350 7500 0    60   ~ 0
 Mir Keyboard\n
@@
 Wire Wire Line
 	5100 3850 5100 4375
-Wire Wire Line
-	2550 1100 2650 1100
-Wire Wire Line
-	2450 1100 2550 1100
-Connection ~ 2550 1100
-Connection ~ 2450 1100
-Connection ~ 2450 3900
-$Comp
-L MCU_Microchip_ATmega:ATmega32U2-AU U1
-U 1 1 5C4CD665
-P 2550 2500
-F 0 "U1" H 2550 1014 50  0000 C CNN
-F 1 "ATmega32U2-AU" H 2550 923 50  0000 C CNN
-F 2 "Housings_DFN_QFN:QFN-32-1EP_5x5mm_Pitch0.5mm" H 2550 2500 50  0001 C CIN
-F 3 "http://ww1.microchip.com/downloads/en/DeviceDoc/doc7799.pdf" H 2550 2500 50  0001 C CNN
-	1    2550 2500
-	1    0    0    -1
-$EndComp
 $Comp
 L Device:Q_NPN_BEC Q1
@@
 $EndComp
 Text GLabel 5100 3325 0    50   Input ~ 0
-RGBLED
-Text GLabel 4875 1600 2    50   Input ~ 0
 RGBLED
 $Comp
@@
 Wire Wire Line
 	9025 2250 10525 2250
-Text GLabel 3250 2600 2    50   Input ~ 0
+Text GLabel 3250 3200 2    50   Input ~ 0
 RGBLED
-Text GLabel 3250 3400 2    50   Input ~ 0
+Text GLabel 3250 2500 2    50   Input ~ 0
 COL1
-Text GLabel 3250 3200 2    50   Input ~ 0
+Text GLabel 3250 2300 2    50   Input ~ 0
 COL3
-Text GLabel 3250 2500 2    50   Input ~ 0
+Text GLabel 3250 3100 2    50   Input ~ 0
 COL2
 Text GLabel 3250 1600 2    50   Input ~ 0
 COL0
+Wire Wire Line
+	1350 1700 1375 1700
+Wire Wire Line
+	1150 1700 1125 1700
+Text GLabel 3250 1400 2    50   Input ~ 0
+ROW0
+$Comp
+L MCU_Microchip_ATmega:ATmega32U2-MU U1
+U 1 1 5D02EA58
+P 2550 2500
+F 0 "U1" H 2550 1011 50  0000 C CNN
+F 1 "ATmega32U2-MU" H 2550 920 50  0000 C CNN
+F 2 "Housings_DFN_QFN:QFN-32-1EP_5x5mm_Pitch0.5mm" H 2550 2500 50  0001 C CIN
+F 3 "http://ww1.microchip.com/downloads/en/DeviceDoc/doc7799.pdf" H 2550 2500 50  0001 C CNN
+	1    2550 2500
+	1    0    0    -1
+$EndComp
+Connection ~ 2450 3900
+Wire Wire Line
+	2550 1100 2650 1100
+Wire Wire Line
+	2550 1100 2450 1100
+Connection ~ 2550 1100
+Connection ~ 2450 1100
 $EndSCHEMATC

Commit message: Finish new PCB
Parts:
- removed CR1, CR2: 0.1u, Capacitors_SMD:C_0603, symbol Device:C_Small
- removed D18, D9: WS2812B, LEDs:LED_WS2812B-PLCC4, symbol LED:WS2812B
- removed Q1: Q_NPN_BEC, TO_SOT_Packages_SMD:SOT-23, symbol Device:Q_NPN_BEC
- removed R10, R27, R7, R8, R9: 1k, Resistors_SMD:R_0805, symbol Device:R_Small
- C1, C2, C3, C4, C5, C6: footprint Capacitors_SMD:C_0603 -> Capacitor_SMD:C_0603_1608Metric
- F1: footprint Fuse_Holders_and_Fuses:Fuse_SMD1206_Reflow -> Fuse:Fuse_1206_3216Metric
- MX1, MX2, MX3, MX4: footprint MX_Alps_Hybrid:MX-1U -> locallib:MXOnly-1U-Hotswap
- R1, R2, R3, R4, R5, R6: footprint Resistors_SMD:R_0805 -> Resistor_SMD:R_0603_1608Metric
- SW1: footprint random-keyboard-parts:Jumper-UserFriendly-Small -> locallib:Alps-SKSV-LargerPads
- U1: footprint Housings_DFN_QFN:QFN-32-1EP_5x5mm_Pitch0.5mm -> locallib:QFN-32-1EP_5x5mm_Pitch0.5mm
- U2: footprint random-keyboard-parts:SOT143B -> locallib:SOT143B
- Y1: footprint Crystals:Crystal_SMD_3225-4pin_3.2x2.5mm -> locallib:Crystal_SMD_3225-4pin_3.2x2.5mm
Connections:
- net RGBLED is gone; now on net COL3: U1.9 (PD3)
- net +5V: no longer MX1.3 (LED), MX2.3 (LED), MX3.3 (LED), MX4.3 (LED)
- net COL0: now also U1.18 (PB4); no longer U1.16 (PB2)
- net COL1: now also U1.19 (PB5); no longer U1.25 (PC5)
- net COL2: now also U1.17 (PB3); no longer U1.8 (PD2)
- net COL3: no longer U1.5 (PC2)
- net ROW0: now also U1.10 (PD4); no longer U1.14 (PB0)
- net at R2.2, USB1.5 (DN2), USB1.7 (DN1): now also U2.2 (IO1); no longer U2.3 (IO2)
- net at R3.1, USB1.6 (DP1), USB1.8 (DP2): now also U2.3 (IO2); no longer U2.2 (IO1)
